Commit message: Corrected mesh paths in URDF file

File: src/so100_robot/urdf/SO_5DOF_ARM100_8j_URDF.SLDASM.urdf (robot description, URDF)
Before this commit: robot SO_5DOF_ARM100_8j_URDF.SLDASM, 7 links, 6 joints
Links:
- link Base: geometry collision mesh filename=package://so100_robot/meshes/Base.STL; visual mesh filename=package://so100_robot/meshes/Base.STL
- link Fixed_Jaw: geometry collision mesh filename=package://so100_robot/meshes/Fixed_Jaw.STL; visual mesh filename=package://so100_robot/meshes/Fixed_Jaw.STL
- link Lower_Arm: geometry collision mesh filename=package://so100_robot/meshes/Lower_Arm.STL; visual mesh filename=package://so100_robot/meshes/Lower_Arm.STL
- link Moving Jaw: geometry collision mesh filename=package://so100_robot/meshes/Moving Jaw.STL; visual mesh filename=package://so100_robot/meshes/Moving Jaw.STL
- link Rotation_Pitch: geometry collision mesh filename=package://so100_robot/meshes/Rotation_Pitch.STL; visual mesh filename=package://so100_robot/meshes/Rotation_Pitch.STL
- link Upper_Arm: geometry collision mesh filename=package://so100_robot/meshes/Upper_Arm.STL; visual mesh filename=package://so100_robot/meshes/Upper_Arm.STL
- link Wrist_Pitch_Roll: geometry collision mesh filename=package://so100_robot/meshes/Wrist_Pitch_Roll.STL; visual mesh filename=package://so100_robot/meshes/Wrist_Pitch_Roll.STL
