Commit message: Fixed mesh paths, lowercased and removed spaces in mesh names to enure mesh loading in Gazebo

File: parta_workspace/src/so_5dof_arm100_8j_urdf_sldasm/urdf/SO_5DOF_ARM100_8j_URDF.SLDASM.urdf (robot description, URDF)
Before this commit: robot SO_5DOF_ARM100_8j_URDF.SLDASM, 7 links, 6 joints
Links:
- link Base: geometry collision mesh filename=package://so_5dof_arm100_8j_urdf_sldasm/meshes/base.STL; visual mesh filename=package://so_5dof_arm100_8j_urdf_sldasm/meshes/base.STL
- link Fixed_Jaw: geometry collision mesh filename=package://so_5dof_arm100_8j_urdf_sldasm/meshes/fixed_jaw.STL; visual mesh filename=package://SO_5DOF_ARM100_8j_URDF.SLDASM/meshes/fixed_jaw.STL
- link Lower_Arm: geometry collision mesh filename=package://so_5dof_arm100_8j_urdf_sldasm/meshes/lower_arm.STL; visual mesh filename=package://so_5dof_arm100_8j_urdf_sldasm/meshes/lower_arm.STL
- link Moving Jaw: geometry collision mesh filename=package://so_5dof_arm100_8j_urdf_sldasm/meshes/moving_jaw.S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; visual mesh filename=package://so_5dof_arm100_8j_urdf_sldasm/meshes/moving_jaw.S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
- link Rotation_Pitch: geometry collision mesh filename=package://so_5dof_arm100_8j_urdf_sldasm/meshes/rotation_pit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; visual mesh filename=package://so_5dof_arm100_8j_urdf_sldasm/meshes/rotation_pit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
- link Upper_Arm: geometry collision mesh filename=package://so_5dof_arm100_8j_urdf_sldasm/meshes/upper_arm.STL; visual mesh filename=package://so_5dof_arm100_8j_urdf_sldasm/meshes/upper_arm.STL
- link Wrist_Pitch_Roll: geometry collision mesh filename=package://so_5dof_arm100_8j_urdf_sldasm/meshes/wrist_pitch_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; visual mesh filename=package://so_5dof_arm100_8j_urdf_sldasm/meshes/wrist_pitch_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
