Commit message: Deleted unnecessary files in root folder to avoid build complications

File: parta_workspace/src/so_5dof_arm100_8j_urdf_sldasm/urdf/so_5dof_arm100_8j_urdf_sldasm.urdf (robot description, URDF)
Before this commit: robot SO_5DOF_ARM100_8j_URDF.SLDASM, 7 links, 6 joints
Links:
- link Fixed_Jaw: geometry collision mesh filename=package://so_5dof_arm100_8j_urdf_sldasm/meshes/fixed_jaw.STL; visual mesh filename=package://so_5dof_arm100_8j_urdf_sldasm/meshes/fixed_jaw.STL

Commit message: Removed ros2_control and gazebo plugin sections from URDF due to crashes

File: parta_workspace/src/so_5dof_arm100_8j_urdf_sldasm/urdf/so_5dof_arm100_8j_urdf_sldasm.urdf (robot description, URDF)
Before this commit: robot so_5dof_arm100_8j_urdf_sldasm, 7 links, 6 joints
Links:
- link Base: geometry collision mesh filename=file:///home/joshua/Desktop/technical-exercise/parta_worksp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; visual mesh filename=file:///home/joshua/Desktop/technical-exercise/parta_worksp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
- link Fixed_Jaw: geometry collision mesh filename=file:///home/joshua/Desktop/technical-exercise/parta_worksp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; visual mesh filename=file:///home/joshua/Desktop/technical-exercise/parta_worksp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
- link Lower_Arm: geometry collision mesh filename=file:///home/joshua/Desktop/technical-exercise/parta_worksp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; visual mesh filename=file:///home/joshua/Desktop/technical-exercise/parta_worksp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
- link Moving Jaw: geometry collision mesh filename=file:///home/joshua/Desktop/technical-exercise/parta_worksp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; visual mesh filename=file:///home/joshua/Desktop/technical-exercise/parta_worksp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
- link Rotation_Pitch: geometry collision mesh filename=file:///home/joshua/Desktop/technical-exercise/parta_worksp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; visual mesh filename=file:///home/joshua/Desktop/technical-exercise/parta_worksp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
- link Upper_Arm: geometry collision mesh filename=file:///home/joshua/Desktop/technical-exercise/parta_worksp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; visual mesh filename=file:///home/joshua/Desktop/technical-exercise/parta_worksp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
- link Wrist_Pitch_Roll: geometry collision mesh filename=file:///home/joshua/Desktop/technical-exercise/parta_worksp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; visual mesh filename=file:///home/joshua/Desktop/technical-exercise/parta_worksp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
